File: H26R00/Design/H26R00.sch (EAGLE design)
At the start: 37 parts, among them P1 HEXABIT_17.32_NO_P6_P7_P12, P2 CON-PHOENIX-350_1751277, P3 CON-PHOENIX-350_1751248, U2 HX711, X1 XTALL_CSTCE8M00G52

Commit message: Adding 3.3V to 5V converter to power the bridge Power the HX711 and bridge from 5V and don't use HX711 regulator
Parts:
- removed C16: 100nF, Hexabitz:C-0603
- removed P2: CON-PHOENIX-350_1751277, Hexabitz:CON-PHOENIX-350_1751277
- removed P3: CON-PHOENIX-350_1751248, Hexabitz:CON-PHOENIX-350_1751248
- removed Q1: (no value), Hexabitz:SEMICON-SMD-IPC_PNP-TRANSISTOR_SOT23
- removed R8, R9: 10K, Hexabitz:R-0603
- added C17: 10uF, Hexabitz:C-0603
- added C18: 1uF, Hexabitz:C-0603
- added S1: CON-PHOENIX-350_1751277, Hexabitz:CON-PHOENIX-350_1751277
- added S2: CON-PHOENIX-350_1751248, Hexabitz:CON-PHOENIX-350_1751248
- added U3: HX711, Hexabitz:HX711
- C10: MPN GRM188R60J106ME84D -> GRM188R61A106KE69D; OCTOPART_URL https://octopart.com/grm188r60j106me84d-murata-29304413?r=s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 -> https://octopart.com/grm188r61a106ke69d-murata-22851381?r=a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; VOLTAGE_RATING 6.3 -> 10V
- D1: value VLMS1300-GS08 -> RED
- U2: value HX711 -> LM2775-Q1; device Hexabitz:HX711 -> Hexabitz:LM2775QDSGRQ1; MFN Avia Semiconductor -> (none); MPN HX711 -> (none)
Connections:
- removed net N$1: C13.1, P2-5.K, Q1.C, R8.2, U2.AVDD
- removed net N$10: C16.2, U2.VBG
- removed net N$11: R8.1, R9.2, U2.VFB
- removed net N$8: Q1.B, U2.BASE
- new net +5V: C10.1, C11.1, C13.1, S1-5.K, U2.VOUT, U3.AVDD, U3.VSUP
- new net N$13: C18.2, U2.C1-
- new net N$3: C18.1, U2.C1+
- net A+: now also S1-2.K; no longer P2-2.K
- net A-: now also S1-3.K; no longer P2-3.K
- net B+: now also S2-2.K; no longer P3-2.K
- net B-: now also S2-1.K; no longer P3-1.K
- net DOUT: now also U3.DOUT; no longer U2.DOUT
- net GND: now also C17.2, S1-1.K, S1-4.K, U2.GND, U2.GND_2, U2.PFM, U3.AGND, U3.VFB, U3.XI; no longer C16.1, P2-1.K, P2-4.K, R9.1, U2.AGND, U2.XI
- net INA+: now also U3.INA+; no longer U2.INA+
- net INA-: now also U3.INA-; no longer U2.INA-
- net INB+: now also U3.INB+; no longer U2.INB+
- net INB-: now also U3.INB-; no longer U2.INB-
- net RATE: now also U3.RATE; no longer U2.RATE
- net SCK: now also U3.PD_SCK; no longer U2.PD_SCK
- net VDD: now also C17.1, U2.EN, U2.OUTDIS, U2.VIN, U3.DVDD; no longer U2.DVDD
- net VDDA: no longer C10.1, C11.1, Q1.E, U2.VSUP
Other:
- note added: "IN+ (5V)"
- note added: "IN- (GND)"
- note removed: "AVDD = 1.25V * (10k+10k) / 10k = 2.5V"
- note removed: "IN+"
- note removed: "IN-"

Commit message: Update BOM Release V0
Parts:
- C13: MPN GRM188R60J106ME84D -> GRM188R61A106KE69D; OCTOPART_URL https://octopart.com/grm188r60j106me84d-murata-29304413?r=s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 -> https://octopart.com/grm188r61a106ke69d-murata-22851381?r=a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; VOLTAGE_RATING 6.3V -> 10V
Other:
- moved on the sheet: C10, C11, C12, C17
Changed lines of the file:
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@@
 <attribute name="CAPACITANCE" value="10uF"/>
 <attribute name="MFN" value="Murata"/>
-<attribute name="MPN" value="GRM188R60J106ME84D"/>
-<attribute name="OCTOPART_URL" value="https://octopart.com/grm188r60j106me84d-murata-29304413?r=sp&amp;s=osVScEPTSN-OxfkF3UyHfg"/>
+<attribute name="MPN" value="GRM188R61A106KE69D"/>
+<attribute name="OCTOPART_URL" value="https://octopart.com/grm188r61a106ke69d-murata-22851381?r=ap&amp;s=o9t4ILLiSny6rfdd0oM5Kg"/>
 <attribute name="TOLERANCE" value="10%"/>
-<attribute name="VOLTAGE_RATING" value="6.3V"/>
+<attribute name="VOLTAGE_RATING" value="10V"/>
 </part>
 <part name="GND9" library="supply1" deviceset="GND" device=""/>
@@
 <attribute name="VALUE" x="177.8" y="78.74" size="1.778" layer="96"/>
 </instance>
-<instance part="C11" gate="G$1" x="127" y="163.83" smashed="yes">
-<attribute name="NAME" x="128.524" y="166.751" size="1.778" layer="95"/>
-<attribute name="VALUE" x="128.524" y="161.671" size="1.778" layer="96"/>
-</instance>
-<instance part="C12" gate="G$1" x="139.7" y="163.83" smashed="yes">
-<attribute name="NAME" x="141.224" y="166.751" size="1.778" layer="95"/>
-<attribute name="VALUE" x="141.224" y="161.671" size="1.778" layer="96"/>
-</instance>
-<instance part="C10" gate="G$1" x="114.3" y="163.83" smashed="yes">
-<attribute name="NAME" x="115.824" y="166.751" size="1.778" layer="95"/>
-<attribute name="VALUE" x="115.824" y="161.671" size="1.778" layer="96"/>
+<instance part="C11" gate="G$1" x="127" y="165.1" smashed="yes">
+<attribute name="NAME" x="128.524" y="168.021" size="1.778" layer="95"/>
+<attribute name="VALUE" x="128.524" y="162.941" size="1.778" layer="96"/>
+</instance>
+<instance part="C12" gate="G$1" x="139.7" y="165.1" smashed="yes">
+<attribute name="NAME" x="141.224" y="168.021" size="1.778" layer="95"/>
+<attribute name="VALUE" x="141.224" y="162.941" size="1.778" layer="96"/>
+</instance>
+<instance part="C10" gate="G$1" x="114.3" y="165.1" smashed="yes">
+<attribute name="NAME" x="115.824" y="168.021" size="1.778" layer="95"/>
+<attribute name="VALUE" x="115.824" y="162.941" size="1.778" layer="96"/>
 </instance>
 <instance part="R4" gate="G$1" x="137.16" y="78.74" smashed="yes" rot="R180">
@@
 <attribute name="VALUE" x="88.9" y="144.78" size="1.778" layer="96"/>
 </instance>
-<instance part="C17" gate="G$1" x="26.67" y="163.83" smashed="yes">
-<attribute name="NAME" x="28.194" y="166.751" size="1.778" layer="95"/>
-<attribute name="VALUE" x="28.194" y="161.671" size="1.778" layer="96"/>
+<instance part="C17" gate="G$1" x="26.67" y="165.1" smashed="yes">
+<attribute name="NAME" x="28.194" y="168.021" size="1.778" layer="95"/>
+<attribute name="VALUE" x="28.194" y="162.941" size="1.778" layer="96"/>
 </instance>
 <instance part="GND18" gate="1" x="26.67" y="147.32" smashed="yes">
@@
 <segment>
 <pinref part="C12" gate="G$1" pin="2"/>
-<wire x1="139.7" y1="161.29" x2="139.7" y2="149.86" width="0.1524" layer="91"/>
+<wire x1="139.7" y1="162.56" x2="139.7" y2="149.86" width="0.1524" layer="91"/>
 <pinref part="GND9" gate="1" pin="GND"/>
 </segment>
@@
 <wire x1="127" y1="149.86" x2="127" y2="156.21" width="0.1524" layer="91"/>
 <pinref part="C10" gate="G$1" pin="2"/>
-<wire x1="127" y1="156.21" x2="127" y2="161.29" width="0.1524" layer="91"/>
-<wire x1="114.3" y1="161.29" x2="114.3" y2="156.21" width="0.1524" layer="91"/>
+<wire x1="127" y1="156.21" x2="127" y2="162.56" width="0.1524" layer="91"/>
+<wire x1="114.3" y1="162.56" x2="114.3" y2="156.21" width="0.1524" layer="91"/>
 <wire x1="114.3" y1="156.21" x2="127" y2="156.21" width="0.1524" layer="91"/>
 <junction x="127" y="156.21"/>
@@
 <pinref part="C17" gate="G$1" pin="2"/>
 <pinref part="GND18" gate="1" pin="GND"/>
-<wire x1="26.67" y1="149.86" x2="26.67" y2="161.29" width="0.1524" layer="91"/>
+<wire x1="26.67" y1="149.86" x2="26.67" y2="162.56" width="0.1524" layer="91"/>
 </segment>
 </net>
@@
 <pinref part="C11" gate="G$1" pin="1"/>
 <pinref part="C10" gate="G$1" pin="1"/>
-<wire x1="127" y1="175.26" x2="127" y2="168.91" width="0.1524" layer="91"/>
-<wire x1="114.3" y1="168.91" x2="114.3" y2="175.26" width="0.1524" layer="91"/>
+<wire x1="127" y1="175.26" x2="127" y2="170.18" width="0.1524" layer="91"/>
+<wire x1="114.3" y1="170.18" x2="114.3" y2="175.26" width="0.1524" layer="91"/>
 <wire x1="114.3" y1="175.26" x2="127" y2="175.26" width="0.1524" layer="91"/>
 <junction x="127" y="175.26"/>
@@
 <segment>
 <pinref part="C12" gate="G$1" pin="1"/>
-<wire x1="139.7" y1="179.07" x2="139.7" y2="168.91" width="0.1524" layer="91"/>
+<wire x1="139.7" y1="179.07" x2="139.7" y2="170.18" width="0.1524" layer="91"/>
 <pinref part="SUPPLY12" gate="G$1" pin="VDD"/>
 </segment>
@@
 <segment>
 <pinref part="C17" gate="G$1" pin="1"/>
-<wire x1="26.67" y1="177.8" x2="26.67" y2="168.91" width="0.1524" layer="91"/>
+<wire x1="26.67" y1="177.8" x2="26.67" y2="170.18" width="0.1524" layer="91"/>
 <pinref part="SUPPLY11" gate="G$1" pin="VDD"/>
 </segment>
