File: H26R01/Design/H26R01.sch (EAGLE design)
At the start: 36 parts, among them P1 HEXABIT_17.32_NO_P6_P7_P12, U2 LM2775-Q1, U3 HX711, X1 XTALL_CSTCE8M00G52

Commit message: - Change the MCU to stm32g0b1ceu6n - Improve the layout design for better performance - Edit the terminal block connectors naming in sch and pcb
Parts:
- removed B, C, D, R: PAD1, Hexabitz:PAD1
- added C16: 100nF, HEXABITZ_RCLS:C-0603
- added C19: 10uF, HEXABITZ_RCLS:C-0603
- added R2: 270R, HEXABITZ_RCLS:R-0603
- added RESET: R, HEXABITZ_USER_INTERFACE_PARTS:PINHD-1X1
- added SWD: (no value), pinhead:PINHD-1X3
- C1: value 10nF -> 100nF; device Hexabitz:C-0603 -> HEXABITZ_RCLS:C-0603; CAPACITANCE 10nF -> (none); MFN KEMET -> (none); MPN C0603C103K5RACTU -> (none); OCTOPART_URL https://octopart.com/c0603c103k5ractu-kemet-133094?r=sp&s=R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 -> (none); TOLERANCE 10% -> (none); VOLTAGE_RATING 50V -> (none)
- C10, C11, C12, C13, C14, C15, C17, C18, C8: device Hexabitz:C-0603 -> HEXABITZ_RCLS:C-0603
- C2: value 1.00uF -> 100nF; device Hexabitz:C-0805-POL -> HEXABITZ_RCLS:C-0603; CAPACITANCE 1.00uF -> (none); MFN Yageo -> (none); MPN CC0805KKX7R7BB105 -> (none); OCTOPART_URL https://octopart.com/cc0805kkx7r7bb105-yageo-8376555?r=sp&s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 -> (none); TOLERANCE 10% -> (none); VOLTAGE_RATING 16V -> (none)
- C3: value 100nF -> 4.7uF; device Hexabitz:C-0603 -> HEXABITZ_RCLS:C-0805-POL; CAPACITANCE 100nF -> (none); MFN KEMET -> (none); MPN C0603C104K8RACTU -> (none); OCTOPART_URL https://octopart.com/c0603c104k8ractu-kemet-145075?r=sp&s=9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 -> (none); TOLERANCE 10% -> (none); VOLTAGE_RATING 10V -> (none)
- C4: value 4.7uF -> 100nF; device Hexabitz:C-0805-POL -> HEXABITZ_RCLS:C-0603; CAPACITANCE 4.7uF -> (none); MFN Murata -> (none); MPN GRM21BC81E475KA12L -> (none); OCTOPART_URL https://octopart.com/grm21bc81e475ka12l-murata-10331911?r=s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 -> (none); TOLERANCE 10% -> (none); VOLTAGE_RATING 25V -> (none)
- C5: value 100nF -> 1uF; device Hexabitz:C-0603 -> HEXABITZ_RCLS:C-0805-POL; CAPACITANCE 100nF -> (none); MFN KEMET -> (none); MPN C0603C104K8RACTU -> (none); OCTOPART_URL https://octopart.com/c0603c104k8ractu-kemet-145075?r=sp&s=9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 -> (none); TOLERANCE 10% -> (none); VOLTAGE_RATING 10 -> (none)
- C6: device Hexabitz:C-0603 -> HEXABITZ_RCLS:C-0603; CAPACITANCE 100nF -> (none); MFN KEMET -> (none); MPN C0603C104K8RACTU -> (none); OCTOPART_URL https://octopart.com/c0603c104k8ractu-kemet-145075?r=sp&s=9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 -> (none); TOLERANCE 10% -> (none); VOLTAGE_RATING 10V -> (none)
- C7: device Hexabitz:C-0805-POL -> HEXABITZ_RCLS:C-0805-POL; CAPACITANCE 4.7uF -> (none); MFN Murata -> (none); MPN GRM21BC81E475KA12L -> (none); OCTOPART_URL https://octopart.com/grm21bc81e475ka12l-murata-10331911?r=s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 -> (none); TOLERANCE 10% -> (none); VOLTAGE_RATING 25V -> (none)
- C9: value 100nF -> 10uF; device Hexabitz:C-0603 -> HEXABITZ_RCLS:C-0603; CAPACITANCE 100nF -> 10uF; MFN KEMET -> Murarta; MPN C0603C104K8RACTU -> GRM188R61A106KE69D; OCTOPART_URL https://octopart.com/c0603c104k8ractu-kemet-145075?r=sp&s=9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 -> https://octopart.com/grm188r61a106ke69d-murata-22851381?r=a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; TOLERANCE 10V -> 10%; VOLTAGE_RATING 10% -> 10V
- FB1: value FB-TDK_MMZ1608Y300B -> (none); device Hexabitz:FB-TDK_MMZ1608Y300B -> HEXABITZ_RCLS:FB-0603; MFN TDK -> (none); MPN MMZ1608Y300B -> (none); OCTOPART_URL https://octopart.com/mmz1608y300b-tdk-368280?r=sp&s=cd9_2ZE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 -> (none)
- R1: value 270.0R -> 0.0R; device Hexabitz:R-0603 -> HEXABITZ_RCLS:R-0603; MFN Yageo -> (none); MPN RC0603FR-07270RL -> (none); OCTOPART_URL https://octopart.com/search?q=RC0603FR-07270RL&start=0 -> (none); RESISTANCE 270.0 Ohm -> (none); TOLERANCE 1% -> (none)
- R3: value 10.0K -> 10K; device Hexabitz:R-0603 -> HEXABITZ_RCLS:R-0603; MFN Yageo -> (none); MPN RC0603JR-0710KL -> (none); OCTOPART_URL https://octopart.com/search?q=RC0603JR-0710KL&start=0 -> (none); RESISTANCE 10.0K Ohm -> (none); TOLERANCE 5% -> (none)
- R4, R5, R6, R7: device Hexabitz:R-0603 -> HEXABITZ_RCLS:R-0603
- S2: device Hexabitz:CON-PHOENIX-350_1751248 -> HEXABITZ_CONNECTION_PARTS:CON-PHOENIX-350_1751248
- U1: value (none) -> STM32G0B1CEU6N; device Hexabitz:STM32F091CBU6 -> HEXABITZ_ICs:STM32G0B1CEU6N
- U2: device Hexabitz:LM2775QDSGRQ1 -> HEXABITZ_ICs:LM2775QDSGRQ1
- U3: device Hexabitz:HX711 -> HEXABITZ_ICs:HX711
Connections:
- removed net B1: B.P$1, R3.2, U1.PF11-OSC_BOOT0
- removed net N$4: D1.A, R1.1
- removed net N$7: D.P$1, U1.PA13
- removed net N$9: C.P$1, U1.PA14
- removed net R1: C8.1, R.P$1, U1.NRST
- new net CLK: R3.2, SWD.1, SWD.2, U1.PA14-BOOT0
- new net DATA: SWD.3, U1.PA13
- new net N$1: D1.A, R2.2
- new net N$8: C1.1, RESET.1, U1.PF2-NRST
- new net VSSA: C10.2, C11.2, C12.2, C13.2, C17.2, C2.2, C3.-, C4.2, C5.-, C8.2, C9.2, R1.1, S1-1.K, S1-4.K, U1.VSS/VSSA, U2.GND, U2.GND_2, U2.PFM, U3.AGND, U3.VFB
- net +5V: now also C8.1, C9.1
- net A+: now also S1-3.K; no longer S1-2.K
- net A-: now also S1-2.K; no longer S1-3.K
- net DOUT: now also U1.PB4; no longer U1.PA10
- net GND: now also C16.2, C19.2, R1.2, U1.EPAD, U1.PB12, U1.PB13, U1.PB14, U1.PB15, U1.VSS; no longer C10.2, C11.2, C12.2, C13.2, C17.2, C2.-, C3.2, C4.-, C5.2, C8.2, C9.2, S1-1.K, S1-4.K, U1.EP, U1.PB5, U1.PB6, U1.PB7, U1.VSS_0, U1.VSS_1, U1.VSS_2, U1.VSS_A, U2.GND, U2.GND_2, U2.PFM, U3.AGND, U3.VFB
- net N$2: now also R2.1, U1.PB2; no longer R1.2, U1.PA11
- net N$5: now also U1.PF1-OSC_OUT; no longer U1.PF0-OSC_IN
- net N$6: now also U1.PF0-OSC_IN; no longer U1.PF1-OSC_OUT
- net RATE: now also U1.PB5; no longer U1.PA6
- net SCK: now also U1.PB3; no longer U1.PA9
- net USART5_RX: now also U1.PD2; no longer U1.PB4
- net USART5_TX: now also U1.PD3; no longer U1.PB3
- net VDD: now also C16.1, C19.1; no longer C12.1, C17.1, C3.1, C4.+, C5.1, C9.1, U1.VBAT, U1.VDD_0, U1.VDD_1, U2.EN, U2.OUTDIS, U2.VIN
- net VDDA: now also C12.1, C17.1, C2.1, C3.+, C4.1, C5.+, U1.VBAT, U1.VDD/VDDA, U1.VREF+, U2.EN, U2.OUTDIS, U2.VIN; no longer C1.1, C2.+, U1.VDDA
Other:
- note added: "5V"
- note added: "BOOT"
- note added: "GND"
- note added: "H26R01"
- note added: "H26R01_Backend"
- note added: "H26R01_Frontend"
- note added: "INA+"
- note added: "INA-"
- note added: "INB+"
- note added: "INB-"
- note added: "Ibrahim Zaeiter"
- note added: "U3 AVDD Coupling"
- note added: "U3 VDD Coupling"
- note added: "VDD\VDDA Coupling"
- note added: "Vref Coupling"
- note removed: "0"
- note removed: "H26R00"
- note removed: "H26R00_Frontend"
- note removed: "I2C1_SCL"
- note removed: "I2C1_SDA"
- note removed: "IN+ (5V)"
- note removed: "IN- (GND)"
- note removed: "OUT+"
- note removed: "OUT-"
- note removed: "VBAT"
- note removed: "VDD Coupling"
- note removed: "VDDA Coupling"
- moved on the sheet: C1, C12, C6, C7, D1, FB1, R1, R3, X1
